Commit message: Add gravity and remove friction

File: simple_models_description/urdf/simple_pmb2.urdf.xacro (robot description, xacro)
@@ -28,4 +28,15 @@
     </inertial>
   </link>
+  <gazebo reference="base_link">
+    <material>Gazebo/White</material>
+    <kp>100000000.0</kp>
+    <kd>10.0</kd>
+    <mu1>0.0</mu1>
+    <mu2>0.0</mu2>
+    <fdir1>1 0 0</fdir1>
+    <maxVel>10.0</maxVel>
+    <minDepth>0.0005</minDepth>
+    <laserRetro>0</laserRetro>
+  </gazebo>
   <link name="base_footprint">
     <visual>
@@ -53,4 +64,15 @@
     </inertial>
   </link>
+  <gazebo reference="base_footprint">
+    <material>Gazebo/White</material>
+    <kp>100000000.0</kp>
+    <kd>10.0</kd>
+    <mu1>0.0</mu1>
+    <mu2>0.0</mu2>
+    <fdir1>1 0 0</fdir1>
+    <maxVel>10.0</maxVel>
+    <minDepth>0.0005</minDepth>
+    <laserRetro>0</laserRetro>
+  </gazebo>
   <joint name="base_footprint_joint" type="fixed">
     <origin xyz="0 0 -0.17" rpy="0 0 0" />
@@ -83,4 +105,15 @@
     </inertial>
   </link>
+  <gazebo reference="base_mid">
+    <material>Gazebo/White</material>
+    <kp>100000000.0</kp>
+    <kd>10.0</kd>
+    <mu1>0.0</mu1>
+    <mu2>0.0</mu2>
+    <fdir1>1 0 0</fdir1>
+    <maxVel>10.0</maxVel>
+    <minDepth>0.0005</minDepth>
+    <laserRetro>0</laserRetro>
+  </gazebo>
   <joint name="base_mid_joint" type="fixed">
     <origin xyz="-0.05 0 0.05" rpy="0 0 0" />
