Commit message: Add velocity and effort limits for pal_local_joint_control

File: simple_models_description/urdf/pendulum.urdf.xacro (robot description, xacro)
@@ -6,5 +6,5 @@
       <child link="pendulum_link"/>
       <dynamics damping="0.01"/>
-      <limit effort="0" velocity="0"/>
+      <limit effort="300.0" velocity="50.0" />
       <safety_controller k_velocity="0"/>
     </joint>
