Commit message: added a box link and joint with transmission for pal physics simulator testing

File: simple_models_description/urdf/box.urdf.xacro (robot description, xacro)
@@ -36,3 +36,45 @@
     </rbdl_contact>
  </link>
+  <link name="box_link">
+    <inertial>
+      <mass value="0.01"/>
+      <inertia ixx="0.04287677484" ixy="0.00043705397" ixz="0.00078292368" iyy="0.03598906971" iyz="0.00037717694" izz="0.01364791564" />
+      <origin rpy="0 0 0" xyz="0.0 0.0 -0.5"/>
+    </inertial>
+    <visual>
+      <origin rpy="0 0 0" xyz="0 0 0"/>
+      <geometry>
+        <cylinder length="0.1" radius="0.00005"/>
+      </geometry>
+      <material name="LightGrey" />
+    </visual>
+    <collision>
+      <origin rpy="0 0 0" xyz="0 0 0"/>
+      <geometry>
+        <cylinder length="0.2" radius="0.00005"/>
+      </geometry>
+      <material name="White" />
+    </collision>
+  </link>
+  <joint name="box_joint" type="prismatic">
+    <parent link="base_link"/>
+    <child link="box_link"/>
+    <origin xyz="0.0 0.0 0.0"
+            rpy="0.0 0.0 0.0"/>
+    <axis xyz="0 0 1" />
+    <limit lower="0" upper="0.2" effort="100.0" velocity="100.0" />
+    <dynamics friction="1.0" damping="1.0"/>
+  </joint>
+  <transmission name="box_joint_trans">
+     <type>transmission_interface/SimpleTransmission</type>
+     <actuator name="box_motor" >
+       <mechanicalReduction> 1.0 </mechanicalReduction>
+     </actuator>
+     <joint name="box_joint">
+       <offset>0.0</offset>
+       <hardwareInterface>hardware_interface/PositionJointInterface</hardwareInterface>
+       <hardwareInterface>hardware_interface/EffortJointInterface</hardwareInterface>
+       <hardwareInterface>hardware_interface/JointStateInterface</hardwareInterface>
+     </joint>
+  </transmission>
 </robot>

Commit message: add transmissions to the simple URDFs

File: simple_models_description/urdf/box.urdf.xacro (robot description, xacro)
@@ -1,4 +1,6 @@
 <?xml version="1.0"?>
 <robot xmlns:xacro="http://ros.org/wiki/xacro">
+  <!--File includes-->
+  <xacro:include filename="$(find simple_models_description)/urdf/transmission.urdf.xacro" />
   <link name="base_link">
     <visual>
@@ -66,15 +68,4 @@
     <dynamics friction="1.0" damping="1.0"/>
   </joint>
-  <transmission name="box_joint_trans">
-     <type>transmission_interface/SimpleTransmission</type>
-     <actuator name="box_motor" >
-       <mechanicalReduction> 1.0 </mechanicalReduction>
-     </actuator>
-     <joint name="box_joint">
-       <offset>0.0</offset>
-       <hardwareInterface>hardware_interface/PositionJointInterface</hardwareInterface>
-       <hardwareInterface>hardware_interface/EffortJointInterface</hardwareInterface>
-       <hardwareInterface>hardware_interface/JointStateInterface</hardwareInterface>
-     </joint>
-  </transmission>
+  <xacro:simple_transmission name="box" reduction="1.0" />
 </robot>

File: simple_models_description/urdf/four_link_chain.urdf.xacro (robot description, xacro)
@@ -1,4 +1,6 @@
 <?xml version="1.0" ?>
 <robot xmlns:xacro="http://ros.org/wiki/xacro">
+    <!--File includes-->
+    <xacro:include filename="$(find simple_models_description)/urdf/transmission.urdf.xacro" />
     <link name="base_link">
         <inertial>
@@ -67,3 +69,6 @@
         </inertial>
     </link>
+    <xacro:simple_transmission name="arm_1" reduction="1.0" />
+    <xacro:simple_transmission name="arm_2" reduction="1.0" />
+    <xacro:simple_transmission name="arm_3" reduction="1.0" />
 </robot>

File: simple_models_description/urdf/four_link_star.urdf.xacro (robot description, xacro)
@@ -1,4 +1,6 @@
 <?xml version="1.0" ?>
 <robot xmlns:xacro="http://ros.org/wiki/xacro">
+    <!--File includes-->
+    <xacro:include filename="$(find simple_models_description)/urdf/transmission.urdf.xacro" />
     <link name="base_link">
         <inertial>
@@ -67,3 +69,6 @@
         </inertial>
     </link>
+    <xacro:simple_transmission name="arm_1" reduction="1.0" />
+    <xacro:simple_transmission name="arm_2" reduction="1.0" />
+    <xacro:simple_transmission name="arm_3" reduction="1.0" />
 </robot>

File: simple_models_description/urdf/pendulum.urdf.xacro (robot description, xacro)
@@ -1,3 +1,6 @@
+<?xml version="1.0"?>
 <robot xmlns:xacro="http://ros.org/wiki/xacro">
+    <!--File includes-->
+    <xacro:include filename="$(find simple_models_description)/urdf/transmission.urdf.xacro" />
     <joint name="pendulum_joint" type="continuous">
       <origin xyz="0 0.18 0.0" rpy="0 0 0"/>
@@ -67,3 +70,4 @@
       </collision>
     </link>
+    <xacro:simple_transmission name="pendulum" reduction="1.0" />
 </robot>
