Commit message: add robot_name and change wheel joint type to fixed in stockbot simple model

File: simple_models_description/urdf/simple_stockbot.urdf.xacro (robot description, xacro)
@@ -1,4 +1,4 @@
 <?xml version="1.0"?>
-<robot xmlns:xacro="http://ros.org/wiki/xacro">
+<robot xmlns:xacro="http://ros.org/wiki/xacro" name="simple_stockbot">
   <xacro:property name="wheel_radius"     value="0.1"/>
   <xacro:property name="wheel_width"      value="0.045"/>
@@ -63,5 +63,5 @@
     </collision>
   </link>
-  <joint name="wheel_left_joint" type="continuous">
+  <joint name="wheel_left_joint" type="fixed">
     <parent link="base_footprint"/>
     <child link="wheel_left_link"/>
@@ -93,5 +93,5 @@
     </collision>
   </link>
-  <joint name="wheel_right_joint" type="continuous">
+  <joint name="wheel_right_joint" type="fixed">
     <parent link="base_footprint"/>
     <child link="wheel_right_link"/>

Commit message: remove stockbot wheels and update mass and origin

File: simple_models_description/urdf/simple_stockbot.urdf.xacro (robot description, xacro)
@@ -13,5 +13,5 @@
     <inertial>
       <origin xyz="-0.00381 0.00312 0.43029" rpy="0 0 0" />
-      <mass value="64.24132" />
+      <mass value="0.1" />
       <inertia ixx="11.896358" ixy="0.001117" ixz="-0.200645"
                iyy="11.897509" iyz="0.11063"
@@ -19,5 +19,5 @@
     </inertial>
     <visual>
-      <origin xyz="0 0 0" rpy="0 0 0" />
+      <origin xyz="0 0 -0.35" rpy="0 0 0" />
       <geometry>
         <mesh filename="package://stockbot_description/meshes/base/base_and_cover.stl" scale="${mesh_scale} ${mesh_scale} ${mesh_scale}"/>
@@ -26,5 +26,5 @@
     </visual>
     <collision>
-      <origin xyz="0 0 0" rpy="0 0 0" />
+      <origin xyz="0 0 -0.35" rpy="0 0 0" />
       <geometry>
         <mesh filename="package://stockbot_description/meshes/base/base_and_cover.stl" scale="${mesh_scale} ${mesh_scale} ${mesh_scale}"/>
@@ -40,63 +40,3 @@
     <parent link="base_link"/>
   </joint>
-  <!-- left wheel -->
-  <link name="wheel_left_link">
-    <inertial>
-      <origin xyz="0 ${0.02086 * -1.0} -0.00259" rpy="0 0 0"/>
-      <mass value="4.31508"/>
-      <inertia ixx="0.013545" ixy="0" ixz="0"
-               iyy="0.010718" iyz="${-0.000921 * -1.0}"
-               izz="0.013395"/>
-    </inertial>
-    <visual>
-      <origin xyz="0 0 0" rpy="0 ${-90 * deg_to_rad} 0"/>
-      <geometry>
-        <mesh filename="package://stockbot_description/meshes/wheels/wheel.stl" scale="0.001 0.001 0.001"/>
-      </geometry>
-      <material name="Grey"/>
-    </visual>
-    <collision>
-      <origin xyz="0 0 0" rpy="0 0 0"/>
-      <geometry>
-        <cylinder radius="${wheel_radius}" length="${wheel_width}"/>
-      </geometry>
-    </collision>
-  </link>
-  <joint name="wheel_left_joint" type="fixed">
-    <parent link="base_footprint"/>
-    <child link="wheel_left_link"/>
-    <origin xyz="0 ${-1.0 * -wheel_separation / 2} 0" rpy="${-90 * -1.0 * deg_to_rad} 0 0"/>
-    <axis xyz="0 0 1"/>
-    <limit effort="${wheel_torque}" velocity="${wheel_velocity / wheel_radius}"/>
-  </joint>
-  <!-- right wheel -->
-  <link name="wheel_right_link">
-    <inertial>
-      <origin xyz="0 ${0.02086 * 1.0} -0.00259" rpy="0 0 0"/>
-      <mass value="4.31508"/>
-      <inertia ixx="0.013545" ixy="0" ixz="0"
-               iyy="0.010718" iyz="${-0.000921 * 1.0}"
-               izz="0.013395"/>
-    </inertial>
-    <visual>
-      <origin xyz="0 0 0" rpy="0 ${-90 * deg_to_rad} 0"/>
-      <geometry>
-        <mesh filename="package://stockbot_description/meshes/wheels/wheel.stl" scale="0.001 0.001 0.001"/>
-      </geometry>
-      <material name="Grey"/>
-    </visual>
-    <collision>
-      <origin xyz="0 0 0" rpy="0 0 0"/>
-      <geometry>
-        <cylinder radius="${wheel_radius}" length="${wheel_width}"/>
-      </geometry>
-    </collision>
-  </link>
-  <joint name="wheel_right_joint" type="fixed">
-    <parent link="base_footprint"/>
-    <child link="wheel_right_link"/>
-    <origin xyz="0 ${1.0 * -wheel_separation / 2} 0" rpy="${-90 * 1.0 * deg_to_rad} 0 0"/>
-    <axis xyz="0 0 1"/>
-    <limit effort="${wheel_torque}" velocity="${wheel_velocity / wheel_radius}"/>
-  </joint>
 </robot>

Commit message: updated simple stockbot urdf xacro

File: simple_models_description/urdf/simple_stockbot.urdf.xacro (robot description, xacro)
@@ -1,40 +1,67 @@
 <?xml version="1.0"?>
 <robot xmlns:xacro="http://ros.org/wiki/xacro" name="simple_stockbot">
-  <xacro:property name="wheel_radius"     value="0.1"/>
-  <xacro:property name="wheel_width"      value="0.045"/>
-  <xacro:property name="wheel_separation" value="0.3517"/>
-  <xacro:property name="wheel_torque"     value="5.5"/>
-  <xacro:property name="wheel_velocity"   value="1.0"/>
   <xacro:property name="deg_to_rad" value="0.01745329251994329577" />
   <xacro:property name="mesh_scale"   value="0.001"/>
-  <!-- Base link -->
-  <xacro:property name="base_link_z" value="0.09877"/>
+  <xacro:property name="base_link_z" value="0.5"/>
+  <xacro:property name="radius" value="0.2"/>
   <link name="base_link">
-    <inertial>
-      <origin xyz="-0.00381 0.00312 0.43029" rpy="0 0 0" />
-      <mass value="0.1" />
-      <inertia ixx="11.896358" ixy="0.001117" ixz="-0.200645"
-               iyy="11.897509" iyz="0.11063"
-               izz="0.796967"/>
-    </inertial>
     <visual>
-      <origin xyz="0 0 -0.35" rpy="0 0 0" />
       <geometry>
         <mesh filename="package://stockbot_description/meshes/base/base_and_cover.stl" scale="${mesh_scale} ${mesh_scale} ${mesh_scale}"/>
       </geometry>
       <material name="DarkGrey" />
+      <origin rpy="0 0 0.1" xyz="0 0 0"/>
     </visual>
     <collision>
-      <origin xyz="0 0 -0.35" rpy="0 0 0" />
       <geometry>
         <mesh filename="package://stockbot_description/meshes/base/base_and_cover.stl" scale="${mesh_scale} ${mesh_scale} ${mesh_scale}"/>
       </geometry>
       <material name="DarkGrey" />
+      <origin rpy="0 0 0.1" xyz="0 0 0"/>
     </collision>
+    <inertial>
+        <origin xyz="0.0 0.0 0.0" rpy="0.0 0.0 0.0" />
+        <mass value="50" />
+         <inertia ixx="0.1"  ixy="0"  ixz="0" iyy="0.1" iyz="0" izz="0.1" />
+    </inertial>
   </link>
-  <!-- Base footprint -->
-  <link name="base_footprint"/>
+  <link name="base_footprint">
+    <visual>
+      <geometry>
+        <cylinder length="0.08" radius="${radius}"/>
+      </geometry>
+      <origin rpy="0 0 0" xyz="0 0 0"/>
+      <material name="blue">
+        <color rgba="0 0 1 1"/>
+      </material>
+    </visual>
+    <collision>
+      <geometry>
+        <cylinder length="0.08" radius="${radius}"/>
+      </geometry>
+      <origin rpy="0 0 0" xyz="0 0 0"/>
+      <material name="blue">
+        <color rgba="0 0 1 1"/>
+      </material>
+    </collision>
+    <inertial>
+        <origin xyz="0.0 0.0 0.0" rpy="0.0 0.0 0.0" />
+        <mass value="50" />
+         <inertia ixx="0.1"  ixy="0"  ixz="0" iyy="0.1" iyz="0" izz="0.1" />
+    </inertial>
+  </link>
+  <gazebo reference="base_footprint">
+    <material>Gazebo/White</material>
+    <kp>100000000.0</kp>
+    <kd>10.0</kd>
+    <mu1>0.0</mu1>
+    <mu2>0.0</mu2>
+    <fdir1>1 0 0</fdir1>
+    <maxVel>10.0</maxVel>
+    <minDepth>0.0005</minDepth>
+    <laserRetro>0</laserRetro>
+  </gazebo>
   <joint name="base_footprint_joint" type="fixed">
-    <origin xyz="0 0 0.09877" rpy="0 0 0" />
+    <origin xyz="0 0 -0.1" rpy="0 0 0" />
     <child link="base_footprint" />
     <parent link="base_link"/>

Commit message: fixed frames order

File: simple_models_description/urdf/simple_stockbot.urdf.xacro (robot description, xacro)
@@ -64,6 +64,6 @@
   <joint name="base_footprint_joint" type="fixed">
     <origin xyz="0 0 -0.1" rpy="0 0 0" />
+    <parent link="base_link"/>
     <child link="base_footprint" />
-    <parent link="base_link"/>
   </joint>
 </robot>

Commit message: Remove rotation of base/cover in simple_stockbot

File: simple_models_description/urdf/simple_stockbot.urdf.xacro (robot description, xacro)
@@ -11,5 +11,5 @@
       </geometry>
       <material name="DarkGrey" />
-      <origin rpy="0 0 0.1" xyz="0 0 0"/>
+      <origin rpy="0 0 0" xyz="0 0 0"/>
     </visual>
     <collision>
@@ -18,5 +18,5 @@
       </geometry>
       <material name="DarkGrey" />
-      <origin rpy="0 0 0.1" xyz="0 0 0"/>
+      <origin rpy="0 0 0" xyz="0 0 0"/>
     </collision>
     <inertial>
