Commit message: Change for muliple pmb2 navigation

File: simple_models_description/robots/robot.urdf.xacro (robot description, xacro)
@@ -7,4 +7,8 @@
     <xacro:wrong_laser_model/>
   </xacro:if>
+  <xacro:arg name="multiple" default="false"/>
+  <xacro:arg name="namespace" default=""/>
+  <xacro:property name="is_multiple" value="$(arg multiple)" />
+  <xacro:property name="nsp" value="$(arg namespace)" />
   <xacro:include filename="$(find simple_models_description)/urdf/$(arg robot).urdf.xacro" />
   <xacro:include filename="$(find simple_models_description)/urdf/sensors.urdf.xacro" />

File: simple_models_description/urdf/gazebo.urdf.xacro (robot description, xacro)
@@ -16,5 +16,12 @@
     <wheelDiameter>0.197</wheelDiameter>
     <torque>6</torque>
-    <commandTopic>nav_vel</commandTopic>
+    <xacro:if value="${is_multiple}">
+      <robotNamespace>/${nsp}</robotNamespace>
+      <commandTopic>/${nsp}/nav_vel</commandTopic>
+    </xacro:if>
+    <xacro:unless value="${is_multiple}">
+      <robotNamespace></robotNamespace>
+      <commandTopic>nav_vel</commandTopic>
+    </xacro:unless>
     <odometryTopic>odom</odometryTopic>
     <odometryFrame>odom</odometryFrame>

File: simple_models_description/urdf/simple_pmb2.urdf.xacro (robot description, xacro)
@@ -2,4 +2,5 @@
 <robot xmlns:xacro="http://ros.org/wiki/xacro">
   <xacro:property name="radius" value="0.27"/>
+  <xacro:property name="small_radius" value="0.22"/>
   <link name="base_link">
     <visual>
@@ -14,5 +15,5 @@
     <collision>
       <geometry>
-        <cylinder length="0.18" radius="${radius}"/>
+        <cylinder length="0.21" radius="${radius}"/>
       </geometry>
       <origin rpy="0 0 0" xyz="0 0 0"/>
@@ -57,3 +58,33 @@
     <parent link="base_link"/>
   </joint>
+  <link name="base_mid">
+    <visual>
+      <geometry>
+        <cylinder length="0.03" radius="${small_radius}"/>
+      </geometry>
+      <origin rpy="0 0 0" xyz="0 0 0"/>
+      <material name="blue">
+        <color rgba="0 0 1 1"/>
+      </material>
+    </visual>
+    <collision>
+      <geometry>
+        <cylinder length="0.03" radius="${small_radius}"/>
+      </geometry>
+      <origin rpy="0 0 0" xyz="0 0 0"/>
+      <material name="blue">
+        <color rgba="0 0 1 1"/>
+      </material>
+    </collision>
+    <inertial>
+        <origin xyz="0.0 0.0 0.0" rpy="0.0 0.0 0.0" />
+        <mass value="50" />
+         <inertia ixx="0.1"  ixy="0"  ixz="0" iyy="0.1" iyz="0" izz="0.1" />
+    </inertial>
+  </link>
+  <joint name="base_mid_joint" type="fixed">
+    <origin xyz="-0.05 0 0.05" rpy="0 0 0" />
+    <child link="base_mid" />
+    <parent link="base_footprint"/>
+  </joint>
 </robot>

Commit message: adapt robot.urdf.xacro according to the robot

File: simple_models_description/robots/robot.urdf.xacro (robot description, xacro)
@@ -2,5 +2,7 @@
 <robot  xmlns:xacro="http://ros.org/wiki/xacro" name="robot" >
   <xacro:arg name="robot" default="simple_pmb2"/>
+  <xacro:arg name="model_name" default="pmb2"/>
   <xacro:arg name="laser_model" default="sick-571"/> <!-- false, hokuyo, sick-551, sick-561, sick-571-->
+  <xacro:property name="robot_model" value="$(arg model_name)" />
   <xacro:property name="laser_model" value="$(arg laser_model)" />
   <xacro:if value="${laser_model not in ['false', False, 'sick-551', 'sick-561', 'sick-571', 'hokuyo']}">
@@ -13,6 +15,12 @@
   <xacro:include filename="$(find simple_models_description)/urdf/$(arg robot).urdf.xacro" />
   <xacro:include filename="$(find simple_models_description)/urdf/sensors.urdf.xacro" />
-  <xacro:include filename="$(find pmb2_description)/gazebo/gazebo.urdf.xacro" />
-  <xacro:include filename="$(find pmb2_description)/urdf/materials.urdf.xacro" />
+  <xacro:if value="${robot_model == 'pmb2'}">
+    <xacro:include filename="$(find pmb2_description)/gazebo/gazebo.urdf.xacro" />
+    <xacro:include filename="$(find pmb2_description)/urdf/materials.urdf.xacro" />
+  </xacro:if>
+  <xacro:if value="${robot_model == 'stockbot'}">
+    <xacro:include filename="$(find stockbot_description)/gazebo/gazebo.urdf.xacro" />
+    <xacro:include filename="$(find stockbot_description)/urdf/materials.urdf.xacro" />
+  </xacro:if>
   <xacro:include filename="$(find simple_models_description)/urdf/gazebo.urdf.xacro" />
   <xacro:base_sensors name="base" laser_model="$(arg laser_model)"/>

Commit message: simplified args and fixed test

File: simple_models_description/robots/robot.urdf.xacro (robot description, xacro)
@@ -2,7 +2,6 @@
 <robot  xmlns:xacro="http://ros.org/wiki/xacro" name="robot" >
   <xacro:arg name="robot" default="simple_pmb2"/>
-  <xacro:arg name="model_name" default="pmb2"/>
   <xacro:arg name="laser_model" default="sick-571"/> <!-- false, hokuyo, sick-551, sick-561, sick-571-->
-  <xacro:property name="robot_model" value="$(arg model_name)" />
+  <xacro:property name="robot_model" value="$(arg robot)" />
   <xacro:property name="laser_model" value="$(arg laser_model)" />
   <xacro:if value="${laser_model not in ['false', False, 'sick-551', 'sick-561', 'sick-571', 'hokuyo']}">
@@ -14,10 +13,10 @@
   <xacro:property name="nsp" value="$(arg namespace)" />
   <xacro:include filename="$(find simple_models_description)/urdf/$(arg robot).urdf.xacro" />
-  <xacro:if value="${robot_model == 'pmb2'}">
+  <xacro:if value="${robot_model == 'simple_pmb2'}">
     <xacro:include filename="$(find pmb2_description)/gazebo/gazebo.urdf.xacro" />
     <xacro:include filename="$(find pmb2_description)/urdf/materials.urdf.xacro" />
     <xacro:include filename="$(find simple_models_description)/urdf/sensors.urdf.xacro" />
   </xacro:if>
-  <xacro:if value="${robot_model == 'stockbot'}">
+  <xacro:if value="${robot_model == 'simple_stockbot'}">
     <xacro:include filename="$(find stockbot_description)/gazebo/gazebo.urdf.xacro" />
     <xacro:include filename="$(find stockbot_description)/urdf/materials.urdf.xacro" />

Commit message: Revert "simplified args and fixed test"
This reverts commit 6c709cacef3b7b4152b9117500792d6eaa0f76c0.

File: simple_models_description/robots/robot.urdf.xacro (robot description, xacro)
@@ -2,6 +2,7 @@
 <robot  xmlns:xacro="http://ros.org/wiki/xacro" name="robot" >
   <xacro:arg name="robot" default="simple_pmb2"/>
+  <xacro:arg name="model_name" default="pmb2"/>
   <xacro:arg name="laser_model" default="sick-571"/> <!-- false, hokuyo, sick-551, sick-561, sick-571-->
-  <xacro:property name="robot_model" value="$(arg robot)" />
+  <xacro:property name="robot_model" value="$(arg model_name)" />
   <xacro:property name="laser_model" value="$(arg laser_model)" />
   <xacro:if value="${laser_model not in ['false', False, 'sick-551', 'sick-561', 'sick-571', 'hokuyo']}">
@@ -13,10 +14,10 @@
   <xacro:property name="nsp" value="$(arg namespace)" />
   <xacro:include filename="$(find simple_models_description)/urdf/$(arg robot).urdf.xacro" />
-  <xacro:if value="${robot_model == 'simple_pmb2'}">
+  <xacro:if value="${robot_model == 'pmb2'}">
     <xacro:include filename="$(find pmb2_description)/gazebo/gazebo.urdf.xacro" />
     <xacro:include filename="$(find pmb2_description)/urdf/materials.urdf.xacro" />
     <xacro:include filename="$(find simple_models_description)/urdf/sensors.urdf.xacro" />
   </xacro:if>
-  <xacro:if value="${robot_model == 'simple_stockbot'}">
+  <xacro:if value="${robot_model == 'stockbot'}">
     <xacro:include filename="$(find stockbot_description)/gazebo/gazebo.urdf.xacro" />
     <xacro:include filename="$(find stockbot_description)/urdf/materials.urdf.xacro" />

Commit message: Ignore model_name in simple_models robot

File: simple_models_description/robots/robot.urdf.xacro (robot description, xacro)
@@ -2,8 +2,10 @@
 <robot  xmlns:xacro="http://ros.org/wiki/xacro" name="robot" >
   <xacro:arg name="robot" default="simple_pmb2"/>
-  <xacro:arg name="model_name" default="pmb2"/>
   <xacro:arg name="laser_model" default="sick-571"/> <!-- false, hokuyo, sick-551, sick-561, sick-571-->
-  <xacro:property name="robot_model" value="$(arg model_name)" />
+  <xacro:property name="robot_model" value="$(arg robot)" />
   <xacro:property name="laser_model" value="$(arg laser_model)" />
+  <xacro:if value="${robot_model not in ['simple_pmb2', 'simple_stockbot']}">
+    <xacro:wrong_robot_model/>
+  </xacro:if>
   <xacro:if value="${laser_model not in ['false', False, 'sick-551', 'sick-561', 'sick-571', 'hokuyo']}">
     <xacro:wrong_laser_model/>
@@ -14,10 +16,10 @@
   <xacro:property name="nsp" value="$(arg namespace)" />
   <xacro:include filename="$(find simple_models_description)/urdf/$(arg robot).urdf.xacro" />
-  <xacro:if value="${robot_model == 'pmb2'}">
+  <xacro:if value="${robot_model == 'simple_pmb2'}">
     <xacro:include filename="$(find pmb2_description)/gazebo/gazebo.urdf.xacro" />
     <xacro:include filename="$(find pmb2_description)/urdf/materials.urdf.xacro" />
     <xacro:include filename="$(find simple_models_description)/urdf/sensors.urdf.xacro" />
   </xacro:if>
-  <xacro:if value="${robot_model == 'stockbot'}">
+  <xacro:if value="${robot_model == 'simple_stockbot'}">
     <xacro:include filename="$(find stockbot_description)/gazebo/gazebo.urdf.xacro" />
     <xacro:include filename="$(find stockbot_description)/urdf/materials.urdf.xacro" />

Commit message: Fixed navigation test with camera_model parameter

File: simple_models_description/robots/robot.urdf.xacro (robot description, xacro)
@@ -12,4 +12,6 @@
   <xacro:property name="is_multiple" value="$(arg multiple)" />
   <xacro:property name="nsp" value="$(arg namespace)" />
+  <xacro:arg name="camera_model" default="structure"/>
+  <xacro:property name="camera_model" value="$(arg camera_model)"/>
   <xacro:include filename="$(find simple_models_description)/urdf/$(arg robot).urdf.xacro" />
   <xacro:if value="${robot_model == 'simple_pmb2'}">

File: simple_models_description/urdf/stockbot_sensors.urdf.xacro (robot description, xacro)
@@ -5,5 +5,6 @@
   <xacro:include filename="$(find stockbot_description)/urdf/sensors/elp_rgb.urdf.xacro"/>
   <xacro:include filename="$(find stockbot_description)/urdf/sensors/structure_sensor.urdf.xacro"/>
-<!--   <xacro:include filename="$(find mynteye_description)/urdf/mynt_eye_d.urdf.xacro"/> -->
+  <xacro:include filename="$(find mynteye_description)/urdf/mynt_eye_d.urdf.xacro"/>
+  <xacro:include filename="$(find realsense2_description)/urdf/_d435.urdf.xacro" />
   <xacro:include filename="$(find stockbot_description)/urdf/base/base_stockbot_calib.urdf.xacro"/>
   <xacro:include filename="$(find stockbot_description)/urdf/base/base_stockbot_default.urdf.xacro"/>
@@ -60,4 +61,6 @@
         rpy="${180 * deg_to_rad} 0 0" />
     </xacro:sick_tim571_laser>
+    <!-- Check which camera model to use -->
+  <xacro:if value="${camera_model == 'structure'}">
     <!-- Depth "base" -->
     <xacro:structure_sensor
@@ -96,4 +99,57 @@
              ${rgb_Y * deg_to_rad}"/>
     </xacro:elp_rgb>
+  </xacro:if>
+  <xacro:if value="${camera_model == 'mynt_eye_d'}">
+    <!-- RGBD -->
+    <xacro:mynteye_d_camera
+      name="base_rgbd_camera"
+      parent="${parent}">
+      <origin
+        xyz="${base_rgbd_x}
+             ${base_rgbd_y}
+             ${base_rgbd_z}"
+        rpy="${base_rgbd_R * deg_to_rad}
+             ${base_rgbd_P * deg_to_rad}
+             ${base_rgbd_Y * deg_to_rad}"/>
+    </xacro:mynteye_d_camera>
+    <xacro:mynteye_d_camera
+      name="roof_rgbd_camera"
+      parent="${parent}">
+      <origin
+        xyz="${roof_rgbd_x}
+             ${roof_rgbd_y}
+             ${roof_rgbd_z}"
+        rpy="${roof_rgbd_R * deg_to_rad}
+             ${roof_rgbd_P * deg_to_rad}
+             ${roof_rgbd_Y * deg_to_rad}"/>
+    </xacro:mynteye_d_camera>
+  </xacro:if>
+  <xacro:if value="${camera_model == 'realsense'}">
+    <!-- RGBD -->
+    <xacro:sensor_d435
+      name="base_rgbd_camera"
+      parent="${parent}_link"
+      topics_ns="base_rgbd_camera">
+      <origin
+        xyz="${base_rgbd_x}
+             ${base_rgbd_y}
+             ${base_rgbd_z}"
+        rpy="${base_rgbd_R * deg_to_rad}
+             ${base_rgbd_P * deg_to_rad}
+             ${base_rgbd_Y * deg_to_rad}"/>
+    </xacro:sensor_d435>
+    <xacro:sensor_d435
+      name="roof_rgbd_camera"
+      parent="${parent}_link"
+      topics_ns="roof_rgbd_camera">
+      <origin
+        xyz="${roof_rgbd_x}
+             ${roof_rgbd_y}
+             ${roof_rgbd_z}"
+        rpy="${roof_rgbd_R * deg_to_rad}
+             ${roof_rgbd_P * deg_to_rad}
+             ${roof_rgbd_Y * deg_to_rad}"/>
+    </xacro:sensor_d435>
+  </xacro:if>
     <!-- IMU -->
     <xacro:imu_sensor
